Commit message: climb working but tom and jerry landing

File: ModelData/LeggedRobot.urdf (robot description, URDF)
Before this commit: robot plane, 13 links, 12 joints
Links:
- added link gripper1, mass 0.241; collision box size=0.1 0.02 0.1; visual box size=0.1 0.02 0.1
- added link gripper2, mass 0.241; collision mesh filename=gripper2.stl scale=1.3 1.3 1; visual mesh filename=gripper2.stl scale=1.3 1.3 1
- added link gripper_base, mass 0.241; collision mesh filename=gripper_base.stl scale=1 1 1; visual mesh filename=gripper_base.stl scale=1 1 1
- added link gripper_lower_arm, mass 0.241; collision mesh filename=gripper_lower_arm.stl scale=1 1 1; visual mesh filename=gripper_lower_arm.stl scale=1 1 1
- added link gripper_upper_arm, mass 0.241; collision mesh filename=gripper_upper_arm.stl scale=1 1 1; visual mesh filename=gripper_upper_arm.stl scale=1 1 1
Joints:
- added joint chassis_gripper_base: type continuous, parent chassis, child gripper_base, origin xyz=0 0.11 0.12 rpy=0 0 0, axis 0 1 0, limit effort=100 velocity=100
- added joint gripper1_gripper2: type continuous, parent gripper1, child gripper2, origin xyz=0.05 0.08 0.01 rpy=0 0 0, axis 1 0 0, limit effort=100 velocity=100
- added joint gripper_base_gripper_lower_arm: type continuous, parent gripper_base, child gripper_lower_arm, origin xyz=-0.03 0.08 0 rpy=0 0 0, axis 1 0 0, limit effort=100 velocity=100
- added joint gripper_lower_arm_gripper_upper_arm: type continuous, parent gripper_lower_arm, child gripper_upper_arm, origin xyz=0 0 -0.33 rpy=0 0 0, axis 1 0 0, limit effort=100 velocity=100
- added joint gripper_upper_arm_gripper1: type continuous, parent gripper_upper_arm, child gripper1, origin xyz=0.03 0.06 0.365 rpy=0 0 0, axis 0 0 1, limit effort=100 velocity=100

Commit message: Complete everything working

File: ModelData/LeggedRobot.urdf (robot description, URDF)
Before this commit: robot plane, 18 links, 17 joints
Links:
- link gripper1: geometry collision mesh filename=Gripper1withBase.stl scale=1 1 1; visual mesh filename=Gripper1withBase.stl scale=1 1 1

File: ModelData/squareDumbell.urdf (robot description, URDF)
Before this commit: robot plane, 3 links, 2 joints
Links:
- link base_link: geometry collision cylinder length=0.5 radius=0.015; visual cylinder length=0.5 radius=0.015
